File: peregrine.kicad_pcb (KiCad board)
At the start: 4 copper layers, 113.2 x 20.4 mm, 49 parts, among them J1 Barrel_Jack, J4 50Ω, SW1 SW_SPDT, SW2 SW_SPDT, U1 MIC5365-3.3YD5, U2 MIC5365-3.3YD5, U3 4020, U4 TS5A3159ADBVR, U5 74AUC1G86, U6 74AUC2G34, X1 ASV-16MHz

Commit message: pcb improvements
todo: sma
Routing:
- net GND: track 44.4 -> 96.4 mm, vias 34 -> 41
- net VCC: track 99.0 -> 130.2 mm, vias 3 -> 6
- net +3V3: track 59.4 -> 74.5 mm
- net FTrig: track 12.4 -> 20.6 mm
- net Net-(R12-Pad2): track 8.88 -> 7.01 mm
- added copper zone on B.Cu, net GND
Other:
- outline, holes or cut-outs redrawn

Commit message: I was doing this too
hm
Parts:
- removed R12: 0, Resistor_SMD:R_0402_1005Metric_Pad0.72x0.64mm_HandSolder
- removed R13: 10kΩ, Resistor_SMD:R_0603_1608Metric_Pad0.98x0.95mm_HandSolder
- removed R14: 10Ω 0.1%, Resistor_SMD:R_0603_1608Metric_Pad0.98x0.95mm_HandSolder
- removed R15: 15Ω 0.1%, Resistor_SMD:R_0603_1608Metric_Pad0.98x0.95mm_HandSolder
- removed the REF** at (138.7, 122.3)
- added D1: PLED, LED_SMD:LED_0603_1608Metric_Pad1.05x0.95mm_HandSolder, F.Cu at (131.5, 98.5)
- added G***: LOGO, QuarterWave:Peregrine, F.Cu at (165.7, 112.2)
- added R10: 15Ω 0.1%, Resistor_SMD:R_0603_1608Metric_Pad0.98x0.95mm_HandSolder, F.Cu at (196.0, 108.6)
- added R6: 0, Resistor_SMD:R_0402_1005Metric_Pad0.72x0.64mm_HandSolder, F.Cu at (133.8, 110.1)
- added R7: 0, Resistor_SMD:R_0402_1005Metric_Pad0.72x0.64mm_HandSolder, F.Cu at (133.8, 111.2)
- added R8: 10kΩ, Resistor_SMD:R_0603_1608Metric_Pad0.98x0.95mm_HandSolder, F.Cu at (151.3, 104.8)
- added R9: 10Ω 0.1%, Resistor_SMD:R_0603_1608Metric_Pad0.98x0.95mm_HandSolder, F.Cu at (192.4, 108.6)
- added REF**: OSHW-Logo2_14.6x12mm_SilkScreen, Symbol:OSHW-Logo2_14.6x12mm_SilkScreen, B.Cu at (126.2, 105.5)
- GND, VIN: moved to B.Cu
- R1: value 0 -> 150Ω; footprint Resistor_SMD:R_0402_1005Metric_Pad0.72x0.64mm_HandSolder -> Resistor_SMD:R_0603_1608Metric_Pad0.98x0.95mm_HandSolder
- moved R1 33.4 mm to (131.5, 96.7), turned to 0 degrees
- moved R2 26.3 mm to (133.8, 105.7)
- moved R3 26.3 mm to (133.8, 106.8)
- moved R4 26.3 mm to (133.8, 107.9)
- moved R5 26.3 mm to (133.8, 109.0)
- moved TP5 25.3 mm to (130.8, 102.8)
- moved C1 25.3 mm to (105.8, 103.1)
- moved C10 25.3 mm to (133.0, 102.7)
- moved C12 25.3 mm to (148.4, 110.7)
- moved C13 25.3 mm to (141.8, 108.8)
- moved C14 25.3 mm to (143.8, 108.8)
- moved C16 25.3 mm to (187.1, 110.9)
- moved C2 25.3 mm to (112.6, 103.1)
- moved C3 25.3 mm to (114.3, 103.1)
- moved C4 25.3 mm to (105.9, 98.1)
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- renumbered Ext. to J2, Ext. to J3, 5 to TP5, 6 to TP6, 7 to TP7, 8 to TP8
Connections:
- R1 pad 1: FTrig -> +3V3
- R1 pad 2: Net-(R1-Pad2) -> Net-(D1-Pad2)
- U3 pad 12: Net-(U3-Pad12) -> Net-(TP6-Pad1)
- U3 pad 13: Net-(U3-Pad13) -> Net-(TP5-Pad1)
- U3 pad 14: Net-(U3-Pad14) -> Net-(TP7-Pad1)
- U3 pad 15: Net-(U3-Pad15) -> Net-(TP8-Pad1)
- U3 pad 4: Net-(R4-Pad2) -> Net-(R5-Pad2)
- U3 pad 5: Net-(R3-Pad2) -> Net-(R4-Pad2)
- U3 pad 6: Net-(R5-Pad2) -> Net-(R6-Pad2)
- U3 pad 7: Net-(R2-Pad2) -> Net-(R3-Pad2)
- U3 pad 9: Net-(R1-Pad2) -> Net-(R2-Pad2)
Routing:
- net Net-(R6-Pad2): track 0.00 -> 4.75 mm
- net Net-(R2-Pad2): track 5.86 -> 1.41 mm, vias 2 -> 0
- net Net-(TP8-Pad1): track 0.00 -> 3.16 mm
- net Net-(U3-Pad15): track 3.16 -> 0.00 mm
- net Net-(D1-Pad2): track 0.00 -> 2.54 mm
- net +3V3: track 74.5 -> 76.9 mm, vias 5 -> 7
- net Net-(R14-Pad1): track 1.78 -> 0.00 mm
- net Net-(R10-Pad2): track 0.00 -> 1.78 mm
- net Net-(R5-Pad2): track 4.75 -> 6.26 mm, vias 0 -> 2
- net Net-(R1-Pad2): track 1.41 -> 0.00 mm
- net Net-(R3-Pad2): track 6.15 -> 5.86 mm, vias 0 -> 2
- net Net-(R4-Pad2): track 6.26 -> 6.13 mm, vias 2 -> 0
- net VCC: vias 6 -> 7
Other:
- board text added: "Ext Pwr."
- board text added: "Ext. Trigger"
- board text added: "GND"
- board text added: "Internal/Ext."
- board text added: "Power"
- board text added: "V+"

Commit message: ready for fab 1
expensive and spooky. yay
Parts:
- removed the C13 at (141.8, 108.8)
- removed the G*** at (161.8, 104.7)
- added C9: 100nF, Capacitor_SMD:C_0603_1608Metric_Pad1.08x0.95mm_HandSolder, F.Cu at (133.0, 102.7)
- added G***: LOGO, QuarterWave:logoWithText12mmMask, F.Cu at (161.8, 104.7)
- C12: value 100nF -> 1μF
- moved C11 26.1 mm to (148.1, 110.7), turned to -90 degrees
- moved C10 9.15 mm to (124.2, 100.1)
- moved TP4 7.38 mm to (139.3, 108.0)
- moved C12 6.85 mm to (141.8, 108.8)
- moved C14 2.28 mm to (181.2, 104.3), turned to -90 degrees
- moved TP3 0.96 mm to (152.2, 107.9)
- renumbered C14 to C13, C15 to C14, C16 to C15, C8 to C7, C9 to C8, VIN to TP1, GND to TP2
Connections:
- C11 pad 1: Net-(C11-Pad1) -> +3V3
- C12 pad 1: +3V3 -> FTrig
- J3 pad 1: Net-(C11-Pad1) -> Net-(C10-Pad1)
- TP5 pad 1: Net-(U3-Pad13) -> Net-(TP5-Pad1)
- TP6 pad 1: Net-(U3-Pad12) -> Net-(TP6-Pad1)
- TP7 pad 1: Net-(U3-Pad14) -> Net-(TP7-Pad1)
- TP8 pad 1: Net-(U3-Pad15) -> Net-(TP8-Pad1)
- U3 pad 11: Net-(C10-Pad1) -> Net-(C9-Pad1)
- U4 pad 1: Net-(C11-Pad1) -> Net-(C10-Pad1)
Routing:
- net Net-(C11-Pad1): track 27.3 -> 0.00 mm, vias 2 -> 0
- net Net-(C10-Pad1): track 3.64 -> 27.3 mm, vias 0 -> 2
- net GND: track 96.5 -> 119.1 mm, vias 41 -> 40
- net Net-(U3-Pad12): track 5.58 -> 0.00 mm
- net Net-(TP6-Pad1): track 0.00 -> 5.58 mm
- net Net-(U3-Pad14): track 5.38 -> 0.00 mm
- net Net-(TP7-Pad1): track 0.00 -> 5.38 mm
- net Net-(C9-Pad1): track 0.00 -> 3.64 mm
- net Net-(U3-Pad13): track 3.37 -> 0.00 mm
- net Net-(TP5-Pad1): track 0.00 -> 3.37 mm
- net VCC: track 130.2 -> 127.6 mm, vias 7 -> 5
- net Trig: track 422.4 -> 420.2 mm
- net FTrig: track 20.6 -> 18.5 mm
- net +3V3: track 76.9 -> 75.8 mm
- net +VDC: track 40.6 -> 39.6 mm
