File: peregrine.kicad_pcb (KiCad board)
At the start: 4 copper layers, 113.2 x 20.4 mm, 52 parts, among them J1 Barrel_Jack, J2 Ext., J3 Ext., J4 50Ω, SW1 SW_SPDT, SW2 SW_SPDT, U1 MIC5365-3.3YD5, U2 MIC5365-3.3YD5, U3 4020, U4 TS5A3159ADBVR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

Commit message: AGH
I always forget that
Other:
- board text added: "JLCJLCJLCJLC"
Changed lines of the file:
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@@
   (gr_arc (start 93 96.413575) (mid 93.585786 94.999361) (end 95 94.413575) (layer "Edge.Cuts") (width 0.1))
   (gr_arc (start 204.2 102.313575) (mid 205.614214 102.899361) (end 206.2 104.313575) (layer "Edge.Cuts") (width 0.1))
+  (gr_text "JLCJLCJLCJLC" (at 99.9 95.7) (layer "B.SilkS")
+    (effects (font (size 1 1) (thickness 0.15)) (justify mirror))
+  )
   (gr_text "GND" (at 97.5 113.713575) (layer "F.SilkS")
     (effects (font (size 1 1) (thickness 0.15)))
