File: peregrine.kicad_pcb (KiCad board)
At the start: 4 copper layers, 113.2 x 20.4 mm, 52 parts, among them J1 Barrel_Jack, J2 Ext., J3 Ext., J4 50Ω, SW1 SW_SPDT, SW2 SW_SPDT, U1 MIC5365-3.3YD5, U2 MIC5365-3.3YD5, U3 4020, U4 TS5A3159ADBVR, U5 74AUC1G86, U6 74AUC2G34, X1 ASV-16MHz

Commit message: this concerns me
i feel like this is not going to be pretty. might need to simulate more
Parts:
- removed the G*** at (161.8, 104.7)
- added G***: LOGO, QuarterWave:logoWithText12mmPartialMask, F.Cu at (153.7, 101.7)
- J4: footprint SMA_RightAngle:SMA-RightAngle -> CONSMA020:LINX_CONSMA020.062-G
- moved R10 14.7 mm to (181.8, 104.6)
- moved R9 14.7 mm to (178.2, 104.6)
- moved C14 14.7 mm to (167.0, 100.4)
- moved C15 14.7 mm to (172.9, 106.9)
- moved U5 14.7 mm to (165.7, 104.6)
- moved U6 14.7 mm to (173.7, 104.6)
- moved G*** 10.4 mm to (158.6, 104.6), turned to -90 degrees
- moved J4 10.4 mm to (192.2, 104.6), turned to 90 degrees
- moved TP3 4.28 mm to (148.6, 105.7)
- moved C12 3.66 mm to (138.9, 106.6)
- moved C13 3.66 mm to (140.9, 106.6)
- moved C11 3.66 mm to (145.2, 108.4)
- moved R8 3.66 mm to (148.4, 102.5)
- moved U4 3.66 mm to (145.0, 104.7)
- moved TP4 3.18 mm to (137.1, 105.7)
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Routing:
- net GND: track 119.1 -> 72.2 mm, vias 40 -> 53
- net VCC: track 127.6 -> 134.0 mm
- net Trig: track 420.2 -> 426.0 mm
- net +VDC: track 39.6 -> 36.1 mm
- net Net-(R8-Pad1): track 11.2 -> 8.60 mm
- net FTrig: track 18.5 -> 16.4 mm
- net Net-(J4-Pad1): track 4.97 -> 6.74 mm
- net +3V3: track 75.8 -> 74.1 mm
- net Net-(C10-Pad1): track 27.3 -> 25.8 mm
Other:
- board size 113.2 x 20.4 mm -> 99.5 x 20.4 mm

Commit message: redesign
why yes i redesigned half of the entire board
Parts:
- removed the C1 at (104.3, 103.1)
- removed the C2 at (111.2, 103.1)
- removed the J2 at (100.2, 109.7)
- removed the SW1 at (109.2, 109.6)
- removed the TP1 at (100.3, 112.4)
- removed the TP2 at (97.7, 112.4)
- removed the U1 at (107.8, 103.1)
- added C10: 10μF, Capacitor_SMD:C_0805_2012Metric_Pad1.18x1.45mm_HandSolder, F.Cu at (108.5, 102.1)
- added C11: 330nF, Capacitor_SMD:C_0805_2012Metric_Pad1.18x1.45mm_HandSolder, F.Cu at (111.9, 102.1)
- added C12: 10μF, Capacitor_SMD:C_0805_2012Metric_Pad1.18x1.45mm_HandSolder, F.Cu at (111.0, 109.7)
- added D1: SMAJ30A, Diode_SMD:D_SMA, F.Cu at (98.0, 108.7)
- added FB1: FerriteBead_Small, Inductor_SMD:L_0603_1608Metric_Pad1.05x0.95mm_HandSolder, F.Cu at (116.8, 107.6)
- added FB2: FerriteBead_Small, Inductor_SMD:L_0603_1608Metric_Pad1.05x0.95mm_HandSolder, F.Cu at (123.1, 104.1)
- added FB3: FerriteBead_Small, Inductor_SMD:L_0603_1608Metric_Pad1.05x0.95mm_HandSolder, F.Cu at (111.1, 107.8)
- added FB4: FerriteBead_Small, Inductor_SMD:L_0603_1608Metric_Pad1.05x0.95mm_HandSolder, F.Cu at (114.6, 98.1)
- added Q1: BSS84, Package_TO_SOT_SMD:SOT-23, F.Cu at (105.4, 102.2)
- added REF**: ESD-Logo_13.2x12mm_SilkScreen, Symbol:ESD-Logo_13.2x12mm_SilkScreen, B.Cu at (168.0, 104.6)
- added TP10: GND, TestPoint:TestPoint_Pad_1.5x1.5mm, F.Cu at (95.8, 111.9)
- added TP9: V+, TestPoint:TestPoint_Pad_1.5x1.5mm, F.Cu at (100.2, 111.9)
- added U5: L78L05_SOT89, Package_TO_SOT_SMD:SOT-89-3, F.Cu at (106.2, 108.2)
- moved REF** 15.9 mm to (140.6, 104.6), turned to 90 degrees
- moved C13 3.55 mm to (111.1, 106.2), turned to 180 degrees
- moved C1 2.60 mm to (116.8, 111.1)
- moved X1 1.55 mm to (121.3, 109.6)
- moved J1 0.99 mm to (95.0, 100.9)
- moved TP7 0.09 mm to (148.5, 105.6)
- renumbered C7 to C1, C3 to C13, C4 to C14, C5 to C15, C6 to C16, C9 to C2, C8 to C3, C12 to C4, C13 to C5, C14 to C6, C15 to C7, C10 to C8, C11 to C9, D1 to D2, J3 to J2, J4 to J3, R2 to R1, R1 to R10, R3 to R2, R4 to R3, R5 to R4, R6 to R5, R7 to R6, R9 to R7, R10 to R8, R8 to R9, SW2 to SW1, TP5 to TP1, TP6 to TP2, TP7 to TP3, TP8 to TP4, TP9 to TP5, TP10 to TP6, TP3 to TP7, TP4 to TP8, U3 to U1, U5 to U2, U6 to U3, U2 to U6
Connections:
- net FTrig renamed /peregrineSelector/FTrig
- net Net-(C10-Pad1) renamed /peregrineSelector/ExtTrig
- net Net-(J4-Pad1) renamed /peregrinePulser/Output
- net Trig renamed /peregrinePulser/Trig
- C1 pad 1: +3V3 -> Net-(C1-Pad1)
- C13 pad 1: VCC -> +5V
- C14 pad 1: +VDC -> +5V
- C15 pad 1: +3V3 -> Net-(C15-Pad1)
- C3 pad 1: +3V3 -> Net-(C3-Pad1)
- C6 pad 2: VCC -> +3V3
- C7 pad 1: VCC -> +3V3
- U1 pad 16: +3V3 -> Net-(C3-Pad1)
- U2 pad 5: VCC -> +3V3
- U3 pad 5: VCC -> +3V3
- U6 pad 1: +VDC -> +5V
- U6 pad 5: +3V3 -> Net-(C15-Pad1)
- X1 pad 1: +3V3 -> Net-(C1-Pad1)
- X1 pad 4: +3V3 -> Net-(C1-Pad1)
Routing:
- net VCC: track 134.0 -> 0.00 mm, vias 5 -> 0
- net +3V3: track 74.1 -> 157.8 mm
- net +5V: track 0.00 -> 43.4 mm, vias 0 -> 5
- net GND: track 72.2 -> 49.3 mm
- net +VDC: track 36.1 -> 20.0 mm
- net PWR: track 13.1 -> 0.00 mm, vias 2 -> 0
- net Net-(C10-Pad1): track 0.00 -> 9.37 mm
- net Net-(C1-Pad1): track 0.00 -> 8.87 mm
- net Net-(C15-Pad1): track 0.00 -> 6.44 mm
- net Net-(C12-Pad1): track 0.00 -> 4.10 mm
- net Net-(C3-Pad1): track 0.00 -> 3.95 mm
- net Net-(R2-Pad2): track 5.71 -> 8.13 mm
Other:
- board text added: "6/18/22"
- board text added: "Ext."
- board text added: "Revision 3"
- board text removed: "Ext Pwr."
- board text removed: "Ext. Trigger"
- board text removed: "GND"
- board text removed: "Internal/Ext."
- board text removed: "Power"
- board text removed: "V+"

Commit message: Production files
i am Afraid
Routing:
- net GND: track 49.3 -> 37.2 mm, vias 53 -> 55
- net +VDC: track 20.0 -> 15.6 mm
Changed lines of the file:
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@@
     (effects (font (size 1 1) (thickness 0.15)))
   )
-  (segment (start 105.41 101.2825) (end 101.885152 101.2825) (width 0.635) (layer "F.Cu") (net 1))
   (segment (start 100.21 111.92) (end 100.21 108.92) (width 0.635) (layer "F.Cu") (net 1))
   (segment (start 101.01 100.92) (end 101.01 106.78863) (width 0.635) (layer "F.Cu") (net 1))
-  (segment (start 101.01 100.92) (end 104.534848 100.92) (width 0.635) (layer "F.Cu") (net 1))
+  (segment (start 105.41 101.2825) (end 101.3725 101.2825) (width 1.016) (layer "F.Cu") (net 1))
+  (segment (start 101.3725 101.2825) (end 101.01 100.92) (width 1.016) (layer "F.Cu") (net 1))
   (arc (start 101.01 106.78863) (mid 100.802086 107.83388) (end 100.21 108.72) (width 0.635) (layer "F.Cu") (net 1))
-  (arc (start 101.885152 101.2825) (mid 101.411523 101.188289) (end 101.01 100.92) (width 0.635) (layer "F.Cu") (net 1))
-  (arc (start 104.534848 100.92) (mid 105.008476 101.014211) (end 105.41 101.2825) (width 0.635) (layer "F.Cu") (net 1))
-  (segment (start 138.93 107.431425) (end 139.943575 107.431425) (width 0.635) (layer "F.Cu") (net 2))
   (segment (start 173.7 103.967893) (end 173.7 102.2) (width 0.29337) (layer "F.Cu") (net 2))
-  (segment (start 144.318575 109.256425) (end 143.43 110.145) (width 0.635) (layer "F.Cu") (net 2))
   (segment (start 172.0625 106.919598) (end 171.982989 106.999109) (width 0.29337) (layer "F.Cu") (net 2))
   (segment (start 170.7 99.2) (end 167.35 99.2) (width 0.29337) (layer "F.Cu") (net 2))
@@
   (segment (start 105.3125 98.125) (end 104.45 98.9875) (width 0.635) (layer "F.Cu") (net 2))
   (segment (start 119.31 113.96) (end 119.31 112.1) (width 0.635) (layer "F.Cu") (net 2))
-  (segment (start 120.21 113.96) (end 119.31 113.96) (width 0.635) (layer "F.Cu") (net 2))
   (segment (start 111.25 98.9875) (end 112.95 98.9875) (width 0.635) (layer "F.Cu") (net 2))
   (segment (start 120.152448 99.287448) (end 119.35 98.485) (width 0.635) (layer "F.Cu") (net 2))
   (segment (start 106.5 98.125) (end 105.3125 98.125) (width 0.635) (layer "F.Cu") (net 2))
-  (segment (start 147.2425 101.618925) (end 146.3575 101.618925) (width 0.635) (layer "F.Cu") (net 2))
   (segment (start 167.35 99.2) (end 167.025 99.525) (width 0.29337) (layer "F.Cu") (net 2))
-  (segment (start 118.41 113.96) (end 120.21 113.96) (width 0.635) (layer "F.Cu") (net 2))
   (segment (start 108.15 98.125) (end 106.5 98.125) (width 0.635) (layer "F.Cu") (net 2))
   (segment (start 165.8 99.5) (end 167 99.5) (width 0.635) (layer "F.Cu") (net 2))
   (segment (start 172.345 104.643575) (end 173.024318 104.643575) (width 0.29337) (layer "F.Cu") (net 2))
-  (segment (start 148.43 101.618925) (end 147.2425 101.618925) (width 0.635) (layer "F.Cu") (net 2))
   (segment (start 143.63 104.731425) (end 142.17 104.731425) (width 0.635) (layer "F.Cu") (net 2))
   (segment (start 122.762551 99.287448) (end 120.152448 99.287448) (width 0.635) (layer "F.Cu") (net 2))
-  (segment (start 144.318575 109.256425) (end 145.23 109.256425) (width 0.635) (layer "F.Cu") (net 2))
   (segment (start 173.377872 104.497128) (end 173.548783 104.326217) (width 0.29337) (layer "F.Cu") (net 2))
-  (segment (start 118.41 113.96) (end 119.31 113.96) (width 0.635) (layer "F.Cu") (net 2))
-  (segment (start 130.412551 111.224562) (end 130.412551 112.687551) (width 0.29337) (layer "F.Cu") (net 2))
   (segment (start 168.447455 108.463575) (end 164.325 108.463575) (width 0.29337) (layer "F.Cu") (net 2))
   (segment (start 167 99.5) (end 167.025 99.525) (width 0.635) (layer "F.Cu") (net 2))
   (segment (start 164.335052 105.293575) (end 164.335052 108.453523) (width 0.29337) (layer "F.Cu") (net 2))
-  (segment (start 139.943575 107.431425) (end 140.93 107.431425) (width 0.635) (layer "F.Cu") (net 2))
   (segment (start 173.695229 103.972664) (end 173.7 103.967893) (width 0.29337) (layer "F.Cu") (net 2))
-  (segment (start 130.412551 112.687551) (end 130.95 113.225) (width 0.29337) (layer "F.Cu") (net 2))
   (via (at 181.510782 111.1) (size 0.8) (drill 0.4) (layers "F.Cu" "B.Cu") (free) (net 2))
   (via (at 150.15 100.35) (size 0.8) (drill 0.4) (layers "F.Cu" "B.Cu") (free) (net 2))
@@
   (via (at 184.9 98.7) (size 0.8) (drill 0.4) (layers "F.Cu" "B.Cu") (free) (net 2))
   (via (at 114.41 100.32) (size 0.8) (drill 0.4) (layers "F.Cu" "B.Cu") (free) (net 2))
+  (via (at 105.41 103.12) (size 0.8) (drill 0.4) (layers "F.Cu" "B.Cu") (free) (net 2))
   (via (at 164.2 95.1) (size 0.8) (drill 0.4) (layers "F.Cu" "B.Cu") (free) (net 2))
   (via (at 123.51 97.92) (size 0.8) (drill 0.4) (layers "F.Cu" "B.Cu") (free) (net 2))
@@
   (via (at 106.5275 109.82) (size 0.8) (drill 0.4) (layers "F.Cu" "B.Cu") (free) (net 2))
   (via (at 171.110782 112.9) (size 0.8) (drill 0.4) (layers "F.Cu" "B.Cu") (free) (net 2))
-  (via (at 146.3575 101.618925) (size 0.8) (drill 0.4) (layers "F.Cu" "B.Cu") (net 2))
+  (via (at 147.21 100.62) (size 0.8) (drill 0.4) (layers "F.Cu" "B.Cu") (net 2))
+  (via (at 106.61 100.82) (size 0.8) (drill 0.4) (layers "F.Cu" "B.Cu") (free) (net 2))
   (via (at 178 97.5) (size 0.8) (drill 0.4) (layers "F.Cu" "B.Cu") (free) (net 2))
+  (via (at 145.21 110.52) (size 0.8) (drill 0.4) (layers "F.Cu" "B.Cu") (free) (net 2))
   (via (at 167.7 95.7) (size 0.8) (drill 0.4) (layers "F.Cu" "B.Cu") (free) (net 2))
   (via (at 113.51 100.32) (size 0.8) (drill 0.4) (layers "F.Cu" "B.Cu") (free) (net 2))
@@
   (via (at 171.1 96.3) (size 0.8) (drill 0.4) (layers "F.Cu" "B.Cu") (free) (net 2))
   (via (at 184.910782 110.5) (size 0.8) (drill 0.4) (layers "F.Cu" "B.Cu") (free) (net 2))
-  (via (at 106.51 101.02) (size 0.8) (drill 0.4) (layers "F.Cu" "B.Cu") (free) (net 2))
   (via (at 105.5275 109.82) (size 0.8) (drill 0.4) (layers "F.Cu" "B.Cu") (free) (net 2))
   (via (at 124.01 98.72) (size 0.8) (drill 0.4) (layers "F.Cu" "B.Cu") (free) (net 2))
@@
   (via (at 105.5275 106.62) (size 0.8) (drill 0.4) (layers "F.Cu" "B.Cu") (free) (net 2))
   (via (at 164.210782 114.1) (size 0.8) (drill 0.4) (layers "F.Cu" "B.Cu") (free) (net 2))
-  (via (at 143.43 110.145) (size 0.8) (drill 0.4) (layers "F.Cu" "B.Cu") (net 2))
+  (via (at 144.01 109.62) (size 0.8) (drill 0.4) (layers "F.Cu" "B.Cu") (net 2))
   (via (at 150.15 107.05) (size 0.8) (drill 0.4) (layers "F.Cu" "B.Cu") (free) (net 2))
   (via (at 131.61 100.32) (size 0.8) (drill 0.4) (layers "F.Cu" "B.Cu") (free) (net 2))
@@
   (via (at 150.15 114.3) (size 0.8) (drill 0.4) (layers "F.Cu" "B.Cu") (free) (net 2))
   (via (at 130.91 99.82) (size 0.8) (drill 0.4) (layers "F.Cu" "B.Cu") (free) (net 2))
-  (via (at 130.95 113.225) (size 0.8) (drill 0.4) (layers "F.Cu" "B.Cu") (net 2))
+  (via (at 130.71 113.02) (size 0.8) (drill 0.4) (layers "F.Cu" "B.Cu") (net 2))
   (via (at 139.943575 107.431425) (size 0.8) (drill 0.4) (layers "F.Cu" "B.Cu") (net 2))
   (via (at 150.15 98.55) (size 0.8) (drill 0.4) (layers "F.Cu" "B.Cu") (free) (net 2))
@@
   )
   (zone (net 2) (net_name "GND") (layer "F.Cu") (hatch edge 0.508)
-    (connect_pads yes (clearance 0))
-    (min_thickness 0.254) (filled_areas_thickness no)
-    (fill yes (thermal_gap 0.508) (thermal_bridge_width 0.508))
-    (polygon
-      (pts
-        (xy 108.05 101.66)
-        (xy 106.39 101.66)
-        (xy 106.39 100.5)
-        (xy 108.05 100.5)
-      )
-    )
-  )
-  (zone (net 2) (net_name "GND") (layer "F.Cu") (hatch edge 0.508)
     (connect_pads (clearance 0))
     (min_thickness 0.254) (filled_areas_thickness no)
@@
         (xy 192.5 99.4)
         (xy 192.5 103.2)
-        (xy 174.32 103.2)
-        (xy 174.32 96.35)
+        (xy 174.22 103.2)
+        (xy 174.22 96.35)
       )
     )
@@
     (polygon
       (pts
-        (xy 174.32 114.8)
+        (xy 174.22 114.8)
         (xy 93 114.8)
         (xy 93 94.4)
-        (xy 174.32 94.4)
+        (xy 174.22 94.4)
       )
     )
@@
     (polygon
       (pts
-        (xy 192.5 109.85)
-        (xy 174.32 112.9)
-        (xy 174.32 106.1)
-        (xy 192.5 106.1)
+        (xy 192.39 109.85)
+        (xy 174.21 112.9)
+        (xy 174.21 106.1)
+        (xy 192.39 106.1)
       )
     )
@@
     (polygon
       (pts
-        (xy 174.32 114.8)
+        (xy 174.22 114.8)
         (xy 93 114.8)
         (xy 93 94.4)
-        (xy 174.32 94.4)
-      )
-    )
+        (xy 174.22 94.4)
+      )
+    )
