File: peregrine.kicad_sch (KiCad schematic)
At the start: 45 parts, among them J1 Barrel_Jack, J1 Ext., J3 50Ω, SW1 SW_SPDT, SW2 SW_SPDT, U1 MIC5365-3.3YD5, U2 MIC5365-3.3YD5, U3 4020, U4 TS5A3159ADBVR, U5 74AUC1G86, U6 74AUC2G34, Y1 16MHz XO

Commit message: footprint changes
get SMA, switches, and barrel tomorrow. am tired
Parts:
- added R15: 15Ω 0.1%, Resistor_SMD:R_0603_1608Metric_Pad0.98x0.95mm_HandSolder, symbol Device:R_Small_US
- C1, C10, C11, C12, C13, C14, C15, C16, C2, C3, C4, C5, C6, C8, C9: footprint (none) -> Capacitor_SMD:C_0603_1608Metric_Pad1.08x0.95mm_HandSolder
- R1, R10, R11, R12, R13, R2, R3, R4, R5, R6, R7, R8, R9: footprint (none) -> Resistor_SMD:R_0603_1608Metric_Pad0.98x0.95mm_HandSolder
- R14: value 25Ω -> 10Ω 0.1%; footprint (none) -> Resistor_SMD:R_0603_1608Metric_Pad0.98x0.95mm_HandSolder
- TP1, TP2: footprint (none) -> TestPoint:TestPoint_Pad_1.5x1.5mm
- TP3, TP4: footprint (none) -> TestPoint:TestPoint_Pad_D1.0mm
- U1, U2: footprint Package_TO_SOT_SMD:SOT-23-5 -> Package_TO_SOT_SMD:SOT-23-5_HandSoldering
- U3: footprint (none) -> Package_SO:TSSOP-20_4.4x5mm_P0.5mm
- U4: footprint Package_TO_SOT_SMD:SOT-23-6 -> Package_TO_SOT_SMD:SOT-23-6_Handsoldering
- U5: footprint (none) -> Package_TO_SOT_SMD:SOT-353_SC-70-5_Handsoldering
- U6: footprint (none) -> Package_TO_SOT_SMD:SOT-363_SC-70-6_Handsoldering
- renumbered J1 to J2
Connections:
- net at R14.1: now also R15.2; no longer J3.1 (In)
- new net: J3.1 (In), R15.1
Other:
- moved on the sheet: J3

Commit message: initial pcb pass
ugh
Parts:
- removed J2: Ext., symbol Connector:Conn_Coaxial
- removed R10, R11, R6, R7, R8, R9: 0, Resistor_SMD:R_0603_1608Metric_Pad0.98x0.95mm_HandSolder, symbol Device:R_Small_US
- removed Y1: 16MHz XO, symbol Device:Crystal_GND23
- added J2, J3: Ext., Connector_PinHeader_2.54mm:PinHeader_1x02_P2.54mm_Vertical, symbol Connector:Conn_01x02_Female
- added TP10: 1.95kHz, TestPoint:TestPoint_Pad_D1.0mm, symbol Connector:TestPoint
- added TP5: 62.5kHz, TestPoint:TestPoint_Pad_D1.0mm, symbol Connector:TestPoint
- added TP6: 31.3kHz, TestPoint:TestPoint_Pad_D1.0mm, symbol Connector:TestPoint
- added TP7: 15.6kHz, TestPoint:TestPoint_Pad_D1.0mm, symbol Connector:TestPoint
- added TP8: 7.81kHz, TestPoint:TestPoint_Pad_D1.0mm, symbol Connector:TestPoint
- added TP9: 3.91kHz, TestPoint:TestPoint_Pad_D1.0mm, symbol Connector:TestPoint
- added X1: ASV-16MHz, Oscillator:Oscillator_SMD_Abracon_ASV-4Pin_7.0x5.1mm, symbol Oscillator:ASV-xxxMHz
- C8: value 100nF -> 10nF
- J1: footprint (none) -> KLDX-0202-A:KLDX-0202-A
- J4: renamed from J3; footprint (none) -> SMA_RightAngle:SMA-RightAngle
- R1, R12, R2, R3, R4, R5: footprint Resistor_SMD:R_0603_1608Metric_Pad0.98x0.95mm_HandSolder -> Resistor_SMD:R_0402_1005Metric_Pad0.72x0.64mm_HandSolder
- SW1, SW2: footprint (none) -> ul_JS102011SCQN:JS102011SCQN
- U3: footprint Package_SO:TSSOP-20_4.4x5mm_P0.5mm -> Package_SO:TSSOP-16_4.4x5mm_P0.65mm
Connections:
- net +2V5 is gone; now on net +3V3: C8.1
- net +3V3: now also X1.1 (EN), X1.4 (Vdd)
- net +VDC: now also J2.1 (Pin_1)
- net GND: now also U1.2 (GND), U2.2 (GND), J2.2 (Pin_2), J3.2 (Pin_2), X1.2 (GND)
- net at U3.13 (Q7): now also TP5.1
- net at C11.1, U4.1: now also J3.1 (Pin_1)
- net at U3.12 (Q8): now also TP6.1
- net at U3.1 (Q11): now also TP9.1
- net at U3.10 (CLK): now also X1.3 (OUT)
- net at U3.14 (Q9): now also TP7.1
- net at U3.15 (Q10): now also TP8.1
- net at U3.2 (Q12): now also TP10.1
Other:
- note added: "1.953125kHz"
- note removed: "1.953125"
- moved on the sheet: C10, C13, C14, C15, C16, C4, C5, C6, C8, C9, J1, J4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

Commit message: I was doing this too
hm
Parts:
- added D1: PLED, LED_SMD:LED_0603_1608Metric_Pad1.05x0.95mm_HandSolder, symbol Device:LED
- added R1: 150Ω, Resistor_SMD:R_0603_1608Metric_Pad0.98x0.95mm_HandSolder, symbol Device:R_Small_US
- renumbered R15 to R10, R1 to R2, R2 to R3, R3 to R4, R4 to R5, R5 to R6, R12 to R7, R13 to R8, R14 to R9
Connections:
- net +3V3: now also R1.1
- net GND: now also D1.1 (K)
- new net: D1.2 (A), R1.2

Commit message: ready for fab 1
expensive and spooky. yay
Parts:
- renumbered C11 to C10, C12 to C11, C13 to C12, C14 to C13, C15 to C14, C16 to C15, C8 to C7, C9 to C8, C10 to C9
Changed lines of the file:
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@@
     (title "Peregrine - Fast Pulse Generator")
     (date "2022-05-29")
-    (rev "2")
+    (rev "3")
     (company "QuarterWave Engineering")
     (comment 1 "Days since last bite: 5")
@@
   (symbol (lib_id "Device:C_Small") (at 125.73 154.94 0) (unit 1)
     (in_bom yes) (on_board yes)
-    (property "Reference" "C13" (id 0) (at 118.11 153.67 0)
+    (property "Reference" "C12" (id 0) (at 118.11 153.67 0)
       (effects (font (size 1.27 1.27)) (justify left))
     )
@@
   (symbol (lib_id "Device:C_Small") (at 133.35 154.94 0) (unit 1)
     (in_bom yes) (on_board yes) (fields_autoplaced)
-    (property "Reference" "C14" (id 0) (at 135.6741 154.1116 0)
+    (property "Reference" "C13" (id 0) (at 135.6741 154.1116 0)
       (effects (font (size 1.27 1.27)) (justify left))
     )
@@
   (symbol (lib_id "Device:C_Small") (at 228.6 53.34 0) (unit 1)
     (in_bom yes) (on_board yes) (fields_autoplaced)
-    (property "Reference" "C11" (id 0) (at 230.9241 52.5116 0)
+    (property "Reference" "C10" (id 0) (at 230.9241 52.5116 0)
       (effects (font (size 1.27 1.27)) (justify left))
     )
@@
   (symbol (lib_id "Device:C_Small") (at 237.49 109.22 90) (unit 1)
     (in_bom yes) (on_board yes) (fields_autoplaced)
-    (property "Reference" "C16" (id 0) (at 237.4963 103.9581 90))
+    (property "Reference" "C15" (id 0) (at 237.4963 103.9581 90))
     (property "Value" "100nF" (id 1) (at 237.4963 106.495 90))
     (property "Footprint" "Capacitor_SMD:C_0603_1608Metric_Pad1.08x0.95mm_HandSolder" (id 2) (at 237.49 109.22 0)
@@
   (symbol (lib_id "Device:C_Small") (at 201.93 113.03 270) (unit 1)
     (in_bom yes) (on_board yes) (fields_autoplaced)
-    (property "Reference" "C15" (id 0) (at 201.9236 107.7681 90))
+    (property "Reference" "C14" (id 0) (at 201.9236 107.7681 90))
     (property "Value" "100nF" (id 1) (at 201.9236 110.305 90))
     (property "Footprint" "Capacitor_SMD:C_0603_1608Metric_Pad1.08x0.95mm_HandSolder" (id 2) (at 201.93 113.03 0)
@@
   (symbol (lib_id "Device:C_Small") (at 31.75 111.76 0) (unit 1)
     (in_bom yes) (on_board yes) (fields_autoplaced)
-    (property "Reference" "C8" (id 0) (at 34.0741 110.9316 0)
+    (property "Reference" "C7" (id 0) (at 34.0741 110.9316 0)
       (effects (font (size 1.27 1.27)) (justify left))
     )
@@
   (symbol (lib_id "Device:C_Small") (at 102.87 106.68 0) (unit 1)
     (in_bom yes) (on_board yes) (fields_autoplaced)
-    (property "Reference" "C9" (id 0) (at 105.1941 105.8516 0)
+    (property "Reference" "C8" (id 0) (at 105.1941 105.8516 0)
       (effects (font (size 1.27 1.27)) (justify left))
     )
@@
   (symbol (lib_id "Device:C_Small") (at 80.01 127 0) (unit 1)
     (in_bom yes) (on_board yes)
-    (property "Reference" "C10" (id 0) (at 73.66 127.0031 0)
+    (property "Reference" "C9" (id 0) (at 73.66 127.0031 0)
       (effects (font (size 1.27 1.27)) (justify left))
     )
@@
   (symbol (lib_id "Device:C_Small") (at 262.89 40.64 0) (unit 1)
     (in_bom yes) (on_board yes) (fields_autoplaced)
-    (property "Reference" "C12" (id 0) (at 265.2141 39.8116 0)
+    (property "Reference" "C11" (id 0) (at 265.2141 39.8116 0)
       (effects (font (size 1.27 1.27)) (justify left))
     )
@@
     )
     (path "/c023f773-00c6-4e18-b8c1-88cedafae761"
-      (reference "C8") (unit 1) (value "10nF") (footprint "Capacitor_SMD:C_0603_1608Metric_Pad1.08x0.95mm_HandSolder")
+      (reference "C7") (unit 1) (value "10nF") (footprint "Capacitor_SMD:C_0603_1608Metric_Pad1.08x0.95mm_HandSolder")
     )
     (path "/c6894b97-4b6b-4998-82bd-1a3a115065e4"
+      (reference "C8") (unit 1) (value "100nF") (footprint "Capacitor_SMD:C_0603_1608Metric_Pad1.08x0.95mm_HandSolder")
+    )
+    (path "/c6f3f1cf-b916-41b4-a3d7-670275b48abc"
       (reference "C9") (unit 1) (value "100nF") (footprint "Capacitor_SMD:C_0603_1608Metric_Pad1.08x0.95mm_HandSolder")
     )
-    (path "/c6f3f1cf-b916-41b4-a3d7-670275b48abc"
+    (path "/97163d7c-cae8-4df5-b010-a7cb3a480faf"
       (reference "C10") (unit 1) (value "100nF") (footprint "Capacitor_SMD:C_0603_1608Metric_Pad1.08x0.95mm_HandSolder")
     )
-    (path "/97163d7c-cae8-4df5-b010-a7cb3a480faf"
+    (path "/ed822ac1-35bd-4743-a00a-26116e7e2c10"
       (reference "C11") (unit 1) (value "100nF") (footprint "Capacitor_SMD:C_0603_1608Metric_Pad1.08x0.95mm_HandSolder")
     )
-    (path "/ed822ac1-35bd-4743-a00a-26116e7e2c10"
-      (reference "C12") (unit 1) (value "100nF") (footprint "Capacitor_SMD:C_0603_1608Metric_Pad1.08x0.95mm_HandSolder")
-    )
     (path "/2f72fdab-c486-485f-a727-cc86ee2c38f4"
-      (reference "C13") (unit 1) (value "1μF") (footprint "Capacitor_SMD:C_0603_1608Metric_Pad1.08x0.95mm_HandSolder")
+      (reference "C12") (unit 1) (value "1μF") (footprint "Capacitor_SMD:C_0603_1608Metric_Pad1.08x0.95mm_HandSolder")
     )
     (path "/479342da-a8e5-4904-8b02-ab91b8ef2566"
+      (reference "C13") (unit 1) (value "100nF") (footprint "Capacitor_SMD:C_0603_1608Metric_Pad1.08x0.95mm_HandSolder")
+    )
+    (path "/addb073d-052c-4ca9-92c5-c416f8d8c862"
       (reference "C14") (unit 1) (value "100nF") (footprint "Capacitor_SMD:C_0603_1608Metric_Pad1.08x0.95mm_HandSolder")
     )
-    (path "/addb073d-052c-4ca9-92c5-c416f8d8c862"
+    (path "/a6b9fc83-f4f3-4f24-917c-147b4d35de79"
       (reference "C15") (unit 1) (value "100nF") (footprint "Capacitor_SMD:C_0603_1608Metric_Pad1.08x0.95mm_HandSolder")
     )
-    (path "/a6b9fc83-f4f3-4f24-917c-147b4d35de79"
-      (reference "C16") (unit 1) (value "100nF") (footprint "Capacitor_SMD:C_0603_1608Metric_Pad1.08x0.95mm_HandSolder")
-    )
     (path "/96448024-5e99-441a-a68e-c824741a1ce8"
